File: esp-prog.sch (KiCad schematic (older format))
At the start: 7 parts, among them J2 Conn_01x17_Socket, J3 Conn_01x17_Socket, J4 Pins_2x10, J5 Pins_2x10, J6 Conn_01x02_Pins

Commit message: Finished layout
Parts:
- gave numbers to parts that had none: 1
- renumbered LED_TARGET_1 to LED2
Changed lines of the file:
@@
 P 3300 1600
 AR Path="/5E5883BD/5E63D6FD" Ref="R?"  Part="1"
-AR Path="/5E63D6FD" Ref="R?"  Part="1"
-F 0 "R?" H 3400 1650 50  0000 L CNN
+AR Path="/5E63D6FD" Ref="R2"  Part="1"
+F 0 "R2" H 3400 1650 50  0000 L CNN
 F 1 "2k" H 3400 1550 50  0000 L CNN
 F 2 "4ms_Resistor:R_0603" V 3230 1600 50  0001 C CNN
@@
 P 3300 1975
 AR Path="/5E5883BD/5E63D703" Ref="D?"  Part="1"
-AR Path="/5E63D703" Ref="LED_TARGET_1"  Part="1"
-F 0 "LED_TARGET_1" V 3375 1825 50  0000 R CNN
+AR Path="/5E63D703" Ref="LED2"  Part="1"
+F 0 "LED2" V 3375 1825 50  0000 R CNN
 F 1 "Blue" V 3275 1825 50  0000 R CNN
 F 2 "4ms_LED:LED_0603_1608Metric" H 3300 1975 50  0001 C CNN
@@
 P 3300 2225
 AR Path="/5E5883BD/5E63D70B" Ref="#PWR?"  Part="1"
-AR Path="/5E63D70B" Ref="#PWR?"  Part="1"
-F 0 "#PWR?" H 3300 1975 50  0001 C CNN
+AR Path="/5E63D70B" Ref="#PWR0121"  Part="1"
+F 0 "#PWR0121" H 3300 1975 50  0001 C CNN
 F 1 "GND" H 3350 2025 50  0000 C CNN
 F 2 "" H 3300 2225 50  0001 C CNN
