File: esp32-pico-kit.sch (KiCad schematic (older format))
At the start: 28 parts, among them J1 USB_B_Micro, Q1 MMS8050, Q2 MMS8050, SW1 SW_PUSH_SMALL, SW2 SW_PUSH_SMALL, U1 AMS1117, U4 CP2102N-A01-GQFN28

Commit message: Finished layout
Parts:
- renumbered D1 to LED1
Changed lines of the file:
@@
 $EndComp
 $Comp
-L Device:LED D1
+L Device:LED LED1
 U 1 1 5E588E17
 P 1500 1725
-F 0 "D1" V 1575 1575 50  0000 R CNN
+F 0 "LED1" V 1575 1575 50  0000 R CNN
 F 1 "Red" V 1475 1575 50  0000 R CNN
 F 2 "4ms_LED:LED_0603_1608Metric" H 1500 1725 50  0001 C CNN
