File: esp-prog.kicad_pcb (KiCad board)
At the start: 2 copper layers, 35.5 x 51.9 mm, 35 parts, among them J1 USB_B_Micro, J2 Conn_01x17_Socket, J3 Conn_01x17_Socket, J4 Pins_2x10, J5 Pins_2x10, J6 Conn_01x02_Pins, Q1 MMS8050, Q2 MMS8050, SW1 SW_PUSH_SMALL, SW2 SW_PUSH_SMALL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

Commit message: few more traces
Routing:
- net /VDD_PICO: track 3.26 -> 20.2 mm, vias 0 -> 3
- net GND: track 54.2 -> 67.1 mm
- net +5V: track 17.9 -> 27.7 mm
Changed lines of the file:
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@@
     (thickness 1.6)
     (drawings 4)
-    (tracks 152)
+    (tracks 191)
     (zones 0)
     (modules 35)
@@
   (segment (start 41.7 53.5) (end 42.2 54) (width 0.25) (layer F.Cu) (net 1))
   (segment (start 39.75 53.5) (end 41.7 53.5) (width 0.25) (layer F.Cu) (net 1))
-  (segment (start 38.723001 53.124999) (end 37.445001 53.124999) (width 0.25) (layer F.Cu) (net 1))
+  (segment (start 32.825 51) (end 32.25 51.575) (width 0.25) (layer F.Cu) (net 1))
+  (segment (start 32.825 49.375) (end 32.825 51) (width 0.25) (layer F.Cu) (net 1))
+  (segment (start 32.900001 48.299999) (end 32.825 48.375) (width 0.25) (layer F.Cu) (net 1))
+  (segment (start 36.050001 48.364999) (end 35.985001 48.299999) (width 0.25) (layer F.Cu) (net 1))
+  (segment (start 36.050001 50.424999) (end 36.050001 48.364999) (width 0.25) (layer F.Cu) (net 1))
+  (segment (start 35.65 50.825) (end 36.050001 50.424999) (width 0.25) (layer F.Cu) (net 1))
+  (segment (start 32.825 48.375) (end 32.825 49.375) (width 0.25) (layer F.Cu) (net 1))
+  (segment (start 35.985001 48.299999) (end 32.900001 48.299999) (width 0.25) (layer F.Cu) (net 1))
+  (segment (start 35.65 51.575) (end 35.65 50.825) (width 0.25) (layer F.Cu) (net 1))
+  (segment (start 35.61 54.316998) (end 35.61 54.96) (width 0.25) (layer F.Cu) (net 1))
+  (segment (start 39.75 53.5) (end 39.098002 53.5) (width 0.25) (layer F.Cu) (net 1))
+  (segment (start 36.801999 53.124999) (end 35.61 54.316998) (width 0.25) (layer F.Cu) (net 1))
   (segment (start 39.098002 53.5) (end 38.723001 53.124999) (width 0.25) (layer F.Cu) (net 1))
-  (segment (start 39.75 53.5) (end 39.098002 53.5) (width 0.25) (layer F.Cu) (net 1))
-  (segment (start 37.445001 53.124999) (end 35.61 54.96) (width 0.25) (layer F.Cu) (net 1))
-  (segment (start 35.61 54.96) (end 34.794999 55.775001) (width 0.25) (layer F.Cu) (net 1))
-  (segment (start 34.794999 55.775001) (end 34.794999 57.474999) (width 0.25) (layer F.Cu) (net 1))
-  (segment (start 34.794999 57.474999) (end 35.58 58.26) (width 0.25) (layer F.Cu) (net 1))
+  (segment (start 38.723001 53.124999) (end 36.801999 53.124999) (width 0.25) (layer F.Cu) (net 1))
+  (segment (start 35.65 52.325) (end 35.65 51.575) (width 0.25) (layer F.Cu) (net 1))
+  (segment (start 36.449999 53.124999) (end 35.65 52.325) (width 0.25) (layer F.Cu) (net 1))
+  (segment (start 36.801999 53.124999) (end 36.449999 53.124999) (width 0.25) (layer F.Cu) (net 1))
+  (segment (start 36.494999 57.345001) (end 35.58 58.26) (width 0.25) (layer F.Cu) (net 1))
+  (segment (start 36.494999 55.909999) (end 36.494999 57.345001) (width 0.25) (layer F.Cu) (net 1))
+  (segment (start 35.61 54.96) (end 36.527499 55.877499) (width 0.25) (layer F.Cu) (net 1))
+  (segment (start 36.527499 55.877499) (end 36.494999 55.909999) (width 0.25) (layer F.Cu) (net 1))
   (segment (start 39.725 55.15) (end 39.725 55.375) (width 0.25) (layer F.Cu) (net 2))
   (segment (start 39.75 55.125) (end 39.725 55.15) (width 0.25) (layer F.Cu) (net 2))
@@
   (segment (start 39.725 55.375) (end 39.75 55.5) (width 0.25) (layer F.Cu) (net 2))
   (segment (start 39.531661 55.568339) (end 39.725 55.375) (width 0.25) (layer F.Cu) (net 2))
+  (segment (start 37.31 54.96) (end 37.918339 55.568339) (width 0.25) (layer F.Cu) (net 2))
+  (segment (start 35.125 50.4) (end 33.95 51.575) (width 0.25) (layer F.Cu) (net 2))
+  (segment (start 35.125 49.375) (end 35.125 50.4) (width 0.25) (layer F.Cu) (net 2))
+  (via (at 37.01 53.99) (size 0.8) (drill 0.4) (layers F.Cu B.Cu) (net 2))
+  (segment (start 37.01 54.66) (end 37.31 54.96) (width 0.25) (layer F.Cu) (net 2))
+  (segment (start 37.01 53.99) (end 37.01 54.66) (width 0.25) (layer F.Cu) (net 2))
+  (segment (start 33.95 52.752062) (end 34.395 53.197062) (width 0.25) (layer F.Cu) (net 2))
+  (via (at 34.395 53.197062) (size 0.8) (drill 0.4) (layers F.Cu B.Cu) (net 2))
+  (segment (start 33.95 51.575) (end 33.95 52.752062) (width 0.25) (layer F.Cu) (net 2))
+  (segment (start 37.01 53.99) (end 35.187938 53.99) (width 0.25) (layer B.Cu) (net 2))
+  (segment (start 35.187938 53.99) (end 34.395 53.197062) (width 0.25) (layer B.Cu) (net 2))
   (segment (start 37.918339 55.568339) (end 39.531661 55.568339) (width 0.25) (layer F.Cu) (net 2))
-  (segment (start 37.31 54.96) (end 37.918339 55.568339) (width 0.25) (layer F.Cu) (net 2))
+  (segment (start 36.32 60.57) (end 36.32 60.8) (width 0.25) (layer F.Cu) (net 2))
+  (via (at 36.32 60.8) (size 0.8) (drill 0.4) (layers F.Cu B.Cu) (net 2))
+  (segment (start 35.6 59.85) (end 36.32 60.57) (width 0.25) (layer F.Cu) (net 2))
+  (segment (start 37.01 53.99) (end 37.04 54.02) (width 0.25) (layer B.Cu) (net 2))
+  (segment (start 37.04 54.02) (end 37.04 60.08) (width 0.25) (layer B.Cu) (net 2))
+  (segment (start 37.04 60.08) (end 36.32 60.8) (width 0.25) (layer B.Cu) (net 2))
   (segment (start 39.05 65.2) (end 38.55 65.2) (width 0.25) (layer F.Cu) (net 3))
   (segment (start 39.980002 65.2) (end 39.05 65.2) (width 0.25) (layer F.Cu) (net 3))
   (segment (start 41.26 63.920002) (end 39.980002 65.2) (width 0.25) (layer F.Cu) (net 3))
   (segment (start 41.26 63.43) (end 41.26 63.920002) (width 0.25) (layer F.Cu) (net 3))
-  (via (at 36.219998 56.75) (size 0.8) (drill 0.4) (layers F.Cu B.Cu) (net 3))
-  (segment (start 36.139998 56.67) (end 36.219998 56.75) (width 0.25) (layer F.Cu) (net 3))
-  (segment (start 35.62 56.67) (end 36.139998 56.67) (width 0.25) (layer F.Cu) (net 3))
-  (segment (start 36.219998 56.75) (end 34.069989 56.75) (width 0.25) (layer B.Cu) (net 3))
-  (via (at 34.069989 56.75) (size 0.8) (drill 0.4) (layers F.Cu B.Cu) (net 3))
-  (segment (start 34.069989 59.630011) (end 33.375 60.325) (width 0.25) (layer F.Cu) (net 3))
-  (segment (start 34.069989 56.75) (end 34.069989 59.630011) (width 0.25) (layer F.Cu) (net 3))
   (segment (start 34.125 60.325) (end 33.375 60.325) (width 0.25) (layer F.Cu) (net 3))
   (segment (start 34.175 60.325) (end 34.125 60.325) (width 0.25) (layer F.Cu) (net 3))
   (segment (start 38.55 64.7) (end 34.175 60.325) (width 0.25) (layer F.Cu) (net 3))
   (segment (start 38.55 65.2) (end 38.55 64.7) (width 0.25) (layer F.Cu) (net 3))
+  (segment (start 37.35 51.575) (end 37.35 51.634998) (width 0.25) (layer F.Cu) (net 3))
+  (segment (start 37.35 50.69) (end 37.39 50.65) (width 0.25) (layer F.Cu) (net 3))
+  (segment (start 37.325 49.375) (end 37.325 49.725) (width 0.25) (layer F.Cu) (net 3))
+  (via (at 37.39 50.65) (size 0.8) (drill 0.4) (layers F.Cu B.Cu) (net 3))
+  (segment (start 37.35 51.575) (end 37.35 50.69) (width 0.25) (layer F.Cu) (net 3))
+  (segment (start 37.325 49.725) (end 37.39 49.79) (width 0.25) (layer F.Cu) (net 3))
+  (segment (start 37.39 49.79) (end 37.39 50.65) (width 0.25) (layer F.Cu) (net 3))
+  (segment (start 33.66999 56.395) (end 34.02499 56.75) (width 0.25) (layer B.Cu) (net 3))
+  (via (at 34.02499 56.75) (size 0.8) (drill 0.4) (layers F.Cu B.Cu) (net 3))
+  (segment (start 34.02499 59.67501) (end 34.02499 56.75) (width 0.25) (layer F.Cu) (net 3))
+  (segment (start 35.83998 50.65) (end 33.66999 52.81999) (width 0.25) (layer B.Cu) (net 3))
+  (segment (start 37.39 50.65) (end 35.83998 50.65) (width 0.25) (layer B.Cu) (net 3))
+  (segment (start 33.375 60.325) (end 34.02499 59.67501) (width 0.25) (layer F.Cu) (net 3))
+  (segment (start 33.66999 52.81999) (end 33.66999 56.395) (width 0.25) (layer B.Cu) (net 3))
+  (segment (start 34.10499 56.67) (end 34.02499 56.75) (width 0.25) (layer F.Cu) (net 3))
+  (segment (start 35.62 56.67) (end 34.10499 56.67) (width 0.25) (layer F.Cu) (net 3))
   (segment (start 33.375 63.55) (end 33.4 63.575) (width 0.25) (layer F.Cu) (net 6))
   (segment (start 33.375 62.025) (end 33.375 63.55) (width 0.25) (layer F.Cu) (net 6))
@@
   (segment (start 39.700011 53.950011) (end 38.500011 53.950011) (width 0.25) (layer F.Cu) (net 10))
   (via (at 38.4 53.85) (size 0.8) (drill 0.4) (layers F.Cu B.Cu) (net 10))
+  (segment (start 37.71874 55.41874) (end 37.71874 54.53126) (width 0.25) (layer B.Cu) (net 10))
+  (segment (start 40.3 60.15) (end 40.3 58) (width 0.25) (layer B.Cu) (net 10))
   (segment (start 37.71874 54.53126) (end 38.4 53.85) (width 0.25) (layer B.Cu) (net 10))
-  (segment (start 37.71874 55.41874) (end 37.71874 54.53126) (width 0.25) (layer B.Cu) (net 10))
   (segment (start 40.3 58) (end 37.71874 55.41874) (width 0.25) (layer B.Cu) (net 10))
-  (segment (start 40.3 60.15) (end 40.3 58) (width 0.25) (layer B.Cu) (net 10))
   (via (at 42.4 60.325) (size 0.8) (drill 0.4) (layers F.Cu B.Cu) (net 11))
   (segment (start 42.4 61.04) (end 42.21 61.23) (width 0.25) (layer F.Cu) (net 11))
@@
   (segment (start 37.28 56.71) (end 37.32 56.67) (width 0.25) (layer F.Cu) (net 69))
   (segment (start 37.28 58.26) (end 37.28 56.71) (width 0.25) (layer F.Cu) (net 69))
+  (segment (start 40.7 56.45) (end 37.54 56.45) (width 0.25) (layer F.Cu) (net 69))
   (segment (start 37.54 56.45) (end 37.32 56.67) (width 0.25) (layer F.Cu) (net 69))
-  (segment (start 40.7 56.45) (end 37.54 56.45) (width 0.25) (layer F.Cu) (net 69))
   (segment (start 42.2 57.55) (end 42.2 56.45) (width 0.25) (layer F.Cu) (net 70))
   (segment (start 42.62 57.97) (end 42.2 57.55) (width 0.25) (layer F.Cu) (net 70))

Commit message: Finished layout
Parts:
- moved J5 23.6 mm to (55.1, 47.0), turned to 180 degrees
- renumbered D1 to LED1, LED_TARGET_1 to LED2
Routing:
- net GND: track 67.1 -> 180.4 mm, vias 0 -> 3
- net /IO0: track 0.00 -> 85.4 mm, vias 0 -> 3
- net /RXD0: track 0.00 -> 50.4 mm, vias 0 -> 1
- net /TXD0: track 0.00 -> 40.7 mm, vias 0 -> 1
- net /EN: track 0.00 -> 36.6 mm, vias 0 -> 1
- net /nRESET: track 0.00 -> 35.5 mm, vias 0 -> 1
- net /VTref: track 0.00 -> 31.0 mm, vias 0 -> 2
- net /TDO: track 0.00 -> 28.2 mm, vias 0 -> 1
- net /TDI: track 0.00 -> 24.3 mm, vias 0 -> 2
- net /TCK: track 0.00 -> 21.4 mm, vias 0 -> 1
- net /VDD_PICO: track 20.2 -> 38.7 mm
- net /TRST_N: track 0.00 -> 18.0 mm, vias 0 -> 1
- net /TMS: track 0.00 -> 15.4 mm, vias 0 -> 1
- net Net-(C7-Pad2): track 0.00 -> 4.39 mm
- net Net-(C6-Pad2): track 0.00 -> 3.81 mm
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Other:
- board text added: "(J-LINK pinout)"
- board text added: "*or fill SMT below*"
- board text added: "*or use JTAG*"
- board text added: "BOOT"
- board text added: "ENABLE"
- board text added: "ESP32-PICO-KIT"
- board text added: "FROM JTAG PROG."
- board text added: "GND"
- board text added: "IO0"
- board text added: "RST"
- board text added: "RXD0"
- board text added: "TCK"
- board text added: "TDI"
- board text added: "TDO"
- board text added: "TMS"
- board text added: "TO ESP32 TARGET"
- board text added: "TXD0"
- board text added: "VT"
- board text added: "VTref"
- board text added: "nRST"
- board text added: "nc"

Commit message: Final cleanup of silk. Created gerbers (oshpark ordered)
Parts:
- added M?: 561-###TAB, 4ms_Hardware:MountingHole_XXXTAB_AdhesiveBase, F.Cu at (60.2, 70.6)
- added M?: 561-###TAB, 4ms_Hardware:MountingHole_XXXTAB_AdhesiveBase, F.Cu at (60.2, 23.9)
- moved LED1 6.23 mm to (32.5, 70.5)
- moved R1 5.71 mm to (32.5, 66.8)
- moved LED2 2.44 mm to (57.2, 70.8), turned to 270 degrees
- moved R2 0.67 mm to (55.7, 70.9), turned to 90 degrees
Routing:
- net +5V: track 27.7 -> 34.2 mm
- net GND: track 180.4 -> 174.1 mm
- net /TDI: track 24.3 -> 22.0 mm
- net Net-(LED2-Pad2): track 1.68 -> 2.22 mm
- net /VTref: track 31.0 -> 31.5 mm
Other:
- board text added: "(SEGGER J-LINK pinout)"
- board text added: "Pico 3.3V to Target"
- board text added: "Target LED"
- board text added: "USB"
- board text removed: "(J-LINK pinout)"
